Commit message: working

File: model/kuka.urdf (robot description, URDF)
Before this commit: robot kuka_lwr, 9 links, 8 joints
Links:
- link kuka_lwr_1_link: geometry collision cylinder length=0.208 radius=0.07; collision sphere radius=0.07
- link kuka_lwr_2_link: geometry collision cylinder length=0.208 radius=0.07; collision sphere radius=0.07
- link kuka_lwr_3_link: geometry collision cylinder length=0.208 radius=0.07; collision sphere radius=0.07
- link kuka_lwr_4_link: geometry collision cylinder length=0.208 radius=0.07; collision sphere radius=0.07
- link kuka_lwr_5_link: geometry collision cylinder length=0.198 radius=0.07; collision sphere radius=0.07
- link kuka_lwr_6_link: geometry collision mesh filename=package://iit-kuka_lwr-ros-pkg/meshes/convex/arm_wrist_conv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; visual mesh filename=package://iit-kuka_lwr-ros-pkg/meshes_arm/arm_wrist.dae
- link kuka_lwr_7_link: geometry collision cylinder length=0.05 radius=0.04; visual mesh filename=package://iit-kuka_lwr-ros-pkg/meshes/link_7.dae
- link kuka_lwr_base_link: geometry collision cylinder length=0.11 radius=0.07; visual mesh filename=package://iit-kuka_lwr-ros-pkg/meshes_arm/arm_base.dae
